Commit message: fix: update elp-camera-ros2-driver subproject commit and add ver1_elp_stereo_camera.urdf.xacro

File: ros2_ws/src/vehicle/jetracer_driver/urdf/ver1_elp_stereo_camera.urdf.xacro (robot description, xacro)
@@ -2,5 +2,5 @@
 <robot name="elp_stereo_camera" xmlns:xacro="http://ros.org/wiki/xacro">
   <xacro:property name="M_PI" value="3.1415926535897931" />
-  <xacro:property name="INTEROCULAR" value="0.0515214" />
+  <xacro:property name="INTEROCULAR" value="0.060" />
   <xacro:property name="BOARD_THICKNESS" value="0.002" />
   <xacro:property name="LENS_LENGTH" value="0.014" />
