Commit message: fix: update camera offsets and add interocular parameters in jetracer launch and URDF files

File: ros2_ws/src/vehicle/jetracer_driver/urdf/elp_stereo_camera.urdf.xacro (robot description, xacro)
@@ -2,8 +2,7 @@
 <robot name="elp_stereo_camera" xmlns:xacro="http://ros.org/wiki/xacro">
   <xacro:property name="M_PI" value="3.1415926535897931" />
-  <xacro:property name="INTEROCULAR" value="0.0515214" />
   <xacro:property name="BOARD_THICKNESS" value="0.002" />
   <xacro:property name="LENS_LENGTH" value="0.014" />
-  <xacro:macro name="elp_stereo_camera" params="name">
+  <xacro:macro name="elp_stereo_camera" params="name interocular:=0.0515214">
     <link name="${name}">
       <visual>
@@ -44,5 +43,5 @@
       <parent link="${name}" />
       <child link="${name}_left_frame" />
-      <origin xyz="${BOARD_THICKNESS/2 + LENS_LENGTH} ${INTEROCULAR/2} 0" />
+      <origin xyz="${BOARD_THICKNESS/2 + LENS_LENGTH} ${interocular/2} 0" />
     </joint>
     <joint name="${name}_left_frame_to_${name}_left_optical_frame" type="fixed">
@@ -54,5 +53,5 @@
       <parent link="${name}" />
       <child link="${name}_right_frame" />
-      <origin xyz="${BOARD_THICKNESS/2 + LENS_LENGTH} ${-INTEROCULAR/2} 0" />
+      <origin xyz="${BOARD_THICKNESS/2 + LENS_LENGTH} ${-interocular/2} 0" />
     </joint>
     <joint name="${name}_right_frame_to_${name}_right_optical_frame" type="fixed">

File: ros2_ws/src/vehicle/jetracer_driver/urdf/jetracer_sensor_kit.urdf.xacro (robot description, xacro)
@@ -17,5 +17,10 @@
   <xacro:arg name="camera_pitch" default="0.0" />
   <xacro:arg name="camera_yaw" default="0.0" />
+  <xacro:arg name="camera_interocular" default="0.05" />
+  <xacro:arg name="camera_mount_to_lens_x" default="0.0" />
+  <xacro:arg name="camera_mount_to_lens_y" default="-0.0075" />
+  <xacro:arg name="camera_mount_to_lens_z" default="0.0" />
   <link name="$(arg base_frame)" />
+  <link name="$(arg camera_frame)_mount" />
   <link name="$(arg lidar_frame)">
     <visual>
@@ -28,5 +33,5 @@
     </visual>
   </link>
-  <xacro:elp_stereo_camera name="$(arg camera_frame)" />
+  <xacro:elp_stereo_camera name="$(arg camera_frame)" interocular="$(arg camera_interocular)" />
   <joint name="$(arg base_frame)_to_$(arg lidar_frame)" type="fixed">
     <parent link="$(arg base_frame)" />
@@ -36,10 +41,17 @@
       rpy="$(arg lidar_roll) $(arg lidar_pitch) $(arg lidar_yaw)" />
   </joint>
-  <joint name="$(arg base_frame)_to_$(arg camera_frame)" type="fixed">
+  <joint name="$(arg base_frame)_to_$(arg camera_frame)_mount" type="fixed">
     <parent link="$(arg base_frame)" />
-    <child link="$(arg camera_frame)" />
+    <child link="$(arg camera_frame)_mount" />
     <origin
       xyz="$(arg camera_x) $(arg camera_y) $(arg camera_z)"
       rpy="$(arg camera_roll) $(arg camera_pitch) $(arg camera_yaw)" />
   </joint>
+  <joint name="$(arg camera_frame)_mount_to_$(arg camera_frame)" type="fixed">
+    <parent link="$(arg camera_frame)_mount" />
+    <child link="$(arg camera_frame)" />
+    <origin
+      xyz="$(arg camera_mount_to_lens_x) $(arg camera_mount_to_lens_y) $(arg camera_mount_to_lens_z)"
+      rpy="0 0 0" />
+  </joint>
 </robot>

Commit message: refactor: unify camera base frame naming to camera_camera_link and simplify URDF and TF alias configurations

File: ros2_ws/src/vehicle/jetracer_driver/urdf/elp_stereo_camera.urdf.xacro (robot description, xacro)
@@ -4,5 +4,7 @@
   <xacro:property name="BOARD_THICKNESS" value="0.002" />
   <xacro:property name="LENS_LENGTH" value="0.014" />
-  <xacro:macro name="elp_stereo_camera" params="name interocular:=0.0515214">
+  <xacro:macro
+    name="elp_stereo_camera"
+    params="name interocular:=0.0515214 left_optical_frame:=camera_infra1_optical_frame right_optical_frame:=camera_infra2_optical_frame">
     <link name="${name}">
       <visual>
@@ -16,47 +18,19 @@
       </visual>
     </link>
-    <link name="${name}_left_frame">
-      <visual>
-        <geometry>
-          <cylinder length="${LENS_LENGTH}" radius="0.005" />
-        </geometry>
-        <origin xyz="${-LENS_LENGTH/2} 0 0" rpy="0 ${M_PI/2} 0" />
-        <material name="black">
-          <color rgba="0 0 0 1" />
-        </material>
-      </visual>
-    </link>
-    <link name="${name}_left_optical_frame" />
-    <link name="${name}_right_frame">
-      <visual>
-        <geometry>
-          <cylinder length="${LENS_LENGTH}" radius="0.005" />
-        </geometry>
-        <origin xyz="${-LENS_LENGTH/2} 0 0" rpy="0 ${M_PI/2} 0" />
-        <material name="black">
-          <color rgba="0 0 0 1" />
-        </material>
-      </visual>
-    </link>
-    <link name="${name}_right_optical_frame" />
-    <joint name="${name}_to_${name}_left_frame" type="fixed">
+    <link name="${left_optical_frame}" />
+    <link name="${right_optical_frame}" />
+    <joint name="${name}_to_${left_optical_frame}" type="fixed">
       <parent link="${name}" />
-      <child link="${name}_left_frame" />
-      <origin xyz="${BOARD_THICKNESS/2 + LENS_LENGTH} ${interocular/2} 0" />
+      <child link="${left_optical_frame}" />
+      <origin
+        xyz="${BOARD_THICKNESS/2 + LENS_LENGTH} ${interocular/2} 0"
+        rpy="${-M_PI/2} 0 ${-M_PI/2}" />
     </joint>
-    <joint name="${name}_left_frame_to_${name}_left_optical_frame" type="fixed">
-      <parent link="${name}_left_frame" />
-      <child link="${name}_left_optical_frame" />
-      <origin xyz="0 0 0" rpy="${-M_PI/2} 0 ${-M_PI/2}" />
-    </joint>
-    <joint name="${name}_to_${name}_right_frame" type="fixed">
+    <joint name="${name}_to_${right_optical_frame}" type="fixed">
       <parent link="${name}" />
-      <child link="${name}_right_frame" />
-      <origin xyz="${BOARD_THICKNESS/2 + LENS_LENGTH} ${-interocular/2} 0" />
-    </joint>
-    <joint name="${name}_right_frame_to_${name}_right_optical_frame" type="fixed">
-      <parent link="${name}_right_frame" />
-      <child link="${name}_right_optical_frame" />
-      <origin xyz="0 0 0" rpy="${-M_PI/2} 0 ${-M_PI/2}" />
+      <child link="${right_optical_frame}" />
+      <origin
+        xyz="${BOARD_THICKNESS/2 + LENS_LENGTH} ${-interocular/2} 0"
+        rpy="${-M_PI/2} 0 ${-M_PI/2}" />
     </joint>
   </xacro:macro>
